File: boards/DM0003/layout/DM0003/layout.kicad_pcb (KiCad board)
At the start: 6 copper layers, 62.1 x 56.2 mm, 82 parts, among them CN1 BM10B-SURS-TF(LF)(SN), IC1 TPD4EUSB30DQAR, IC10 ?, IC2 TPD4EUSB30DQAR, IC3 STMPS2151STR, IC4 SN74LVC1G14DRLRG4, IC5 AP3441SHE-7B, IC6 AP22653W6-7, IC7 TPD4EUSB30DQAR, IC8 TPD4EUSB30DQAR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

Commit message: update layout
Parts:
- IC10: value ? -> TUSB321RWBR
