File: boards/DM0003/layout/DM0003/layout.kicad_pcb (KiCad board)
At the start: 6 copper layers, 62.1 x 56.2 mm, 82 parts, among them CN1 BM10B-SURS-TF(LF)(SN), IC1 TPD4EUSB30DQAR, IC10 TUSB321RWBR, IC2 TPD4EUSB30DQAR, IC3 STMPS2151STR, IC4 SN74LVC1G14DRLRG4, IC5 AP3441SHE-7B, IC6 AP22653W6-7, IC7 TPD4EUSB30DQAR, IC8 TPD4EUSB30DQAR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

Commit message: pass drc no unconnected nets + bom matched
Parts:
- C6: value 4.7nF 16V X5R -> GRM155R71H472KA01D
- IC4: value SN74LVC1G14DRLRG4 -> SN74LVC1G14DRLR
- USB1: value HDMI-101S -> 685119248123
- Y1: value ASEK-32.768KHZ-L-R-T -> ASEK-32.768KHZ-LRT
- renumbered U2 to IC10, IC10 to IC11
