File: boards/DM0003/layout/DM0003/layout.kicad_pcb (KiCad board)
At the start: 6 copper layers, 62.1 x 56.2 mm, 82 parts, among them CN1 BM10B-SURS-TF(LF)(SN), IC1 TPD4EUSB30DQAR, IC10 HD3SS3212IRKSR, IC11 TUSB321RWBR, IC2 TPD4EUSB30DQAR, IC3 STMPS2151STR, IC4 SN74LVC1G14DRLR, IC5 AP3441SHE-7B, IC6 AP22653W6-7, IC7 TPD4EUSB30DQAR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

Commit message: chore(DM0003): update layout
Parts:
- moved C21 0.50 mm to (57.1, 61.5)
- moved C22 0.50 mm to (57.1, 67.1)
- moved D5 0.50 mm to (58.2, 64.3)
- moved J10 0.50 mm to (51.8, 64.3)
- moved R18 0.50 mm to (66.5, 85.2)
Routing:
- net 5V: track 22.3 -> 21.7 mm
