File: boards/DM0001/src/layout/HallEncoder/layout.kicad_pcb (KiCad board)
At the start: 2 copper layers, 14 parts, among them J1 BM05B-SRSS-TB

Commit message: Sync reference design layouts
Parts:
- C1, C2, C3: value 10pF 10V -> GCM1555C1H100FA16D
- C4: value 100nF 16V X7R -> GCM155R71H104KE02D
- J1: value BM05B-SRSS-TB -> BM05B-SRSS-TB(LF)(SN)
- R1, R2, R3, R4, R5, R6: value 10k -> ERJ-2RKF1002X
