File: boards/DM0001/src/layout/PhaseDriver_Long/layout.kicad_pcb (KiCad board)
At the start: 2 copper layers, 19 parts, among them U1 STL180N6F7, U2 STL180N6F7, U3 L6387ED

Commit message: remove ignored files
Parts:
- renumbered U3 to IC1, U1 to Q1, U2 to Q2

Commit message: Sync reference design layouts
Parts:
- C1: value 1nF 100V -> GRM1885C1H102JA01D
- C2: value 1uF 25V -> GCM188R71E105KA64D
- C3, C4: value 100pF 10V -> GCM1555C1H101FA16D
- C5: value 470nF 16V -> CL10A474KA8NNNC
- R1: value 2.2k -> ERJ-2RKF2201X
- R2, R4: value 33 -> ERJ-3EKF33R0V
- R3, R5: value 10k -> ERJ-2RKF1002X
- R6: value 10k -> ERJ-3EKF1002V
- R7: value 1 -> RC0805JR-071RL
- R8: value 3m 1% -> CSNL2512FT3L00
