File: boards/DM0003/src/layout_Ethernet/layout.kicad_pcb (KiCad board)
At the start: 2 copper layers, 6 parts, among them IC1 TPD4EUSB30DQAR, IC2 TPD4EUSB30DQAR, J1 CRJ009-ML4-TH

Commit message: Sync layouts (#61)
* Sync reference design layouts

* Remove stale properties

* Update board layouts
Parts:
- R1: value 0 -> ERJ-2GE0R00X
- R2, R3: value 470 -> ERJ-2RKF4700X
Connections:
- net N2857 renamed ETH.NC_CRJ009-ML4-TH_NC_1
- net N2858 renamed ETH.NC_CRJ009-ML4-TH_NC_2
- net io_3v3pi renamed 3V3PI
- net io_gnd renamed GND
- net k_green renamed K_GREEN
- net k_yellow renamed K_YELLOW
- net mp renamed MP
- net nLed_G renamed NLED_G
- net nLed_Y renamed NLED_Y
