File: reference/AP3441x/layout_ap3441x/layout.kicad_pcb (KiCad board)
At the start: 2 copper layers, 9 parts, among them U1 AP3441SHE-7B, U2 XAL5030-222MEC

Commit message: Sync layouts (#61)
* Sync reference design layouts

* Remove stale properties

* Update board layouts
Parts:
- C1: value 4.7nF 16V X5R -> GRM155R71H472KA01D
- C2: value 10uF 16V X7R -> GRM21BZ71E106KE15K
- C3, C5: value 100nF 16V X7R -> GCM155R71H104KE02D
- C4: value 10uF 16V X5R -> GRM21BZ71E106KE15K
- R1: value 10k -> ERJ-2RKF1002X
- R2: value 45.3k -> ERJ-2RKF4532X
- renumbered U1 to IC1, U2 to L1
Connections:
- net enable renamed ENABLE
- net fb_node renamed FB_NODE
- net gnd renamed GND
- net lx_out renamed LX_OUT
- net nc renamed AP3441SHEM7B.NC_AP3441SHE-7B_NC
- net pg renamed PG
- net vin renamed VIN
- net vout renamed VOUT
