File: reference/RP_CM5_IO/Layout_CM5IO/layout.kicad_pcb (KiCad board)
At the start: 2 copper layers, 6 parts, among them U1 10164227-1001A1RLF, U2 10164227-1001A1RLF

Commit message: fix mounting holes
Parts:
- H1, H2, H3, H4: value M2.5 DIN965 Mechanical -> M2.5 DIN965 Via
- renumbered U1 to J1, U2 to J2

Commit message: Sync layouts (#61)
* Sync reference design layouts

* Remove stale properties

* Update board layouts
Parts:
- H1, H2, H3, H4: value M2.5 DIN965 Via -> M2.5 DIN965 Mechanical
Connections:
- net BT_nDisable renamed BT_NDISABLE
- net EEPROM_nWP renamed EEPROM_NWP
- net Ethernet_Pair0_N renamed ETHERNET_PAIR0_N
- net Ethernet_Pair0_P renamed ETHERNET_PAIR0_P
- net Ethernet_Pair1_N renamed ETHERNET_PAIR1_N
- net Ethernet_Pair1_P renamed ETHERNET_PAIR1_P
- net Ethernet_Pair2_N renamed ETHERNET_PAIR2_N
- net Ethernet_Pair2_P renamed ETHERNET_PAIR2_P
- net Ethernet_Pair3_N renamed ETHERNET_PAIR3_N
- net Ethernet_Pair3_P renamed ETHERNET_PAIR3_P
- net Ethernet_SYNC_OUT_3V3 renamed ETHERNET_SYNC_OUT_3V3
- net Ethernet_nLED2_3V3 renamed ETHERNET_NLED2_3V3
- net Ethernet_nLED3_3V3 renamed ETHERNET_NLED3_3V3
- net GPIO_VREF_1V8_3V3_Input renamed GPIO_VREF_1V8_3V3_INPUT
- net LED_nACT renamed LED_NACT
- net LED_nPWR renamed LED_NPWR
- net PCIE_nWAKE renamed PCIE_NWAKE
- net PCIe_CLK_N renamed PCIE_CLK_N
- net PCIe_CLK_P renamed PCIE_CLK_P
- net PCIe_RX_N renamed PCIE_RX_N
- net PCIe_RX_P renamed PCIE_RX_P
- net PCIe_TX_N renamed PCIE_TX_N
- net PCIe_TX_P renamed PCIE_TX_P
- net PCIe_nCLKREQ renamed PCIE_NCLKREQ
- net PCIe_nRST renamed PCIE_NRST
- net SD_VDD_Override renamed SD_VDD_OVERRIDE
- net V1V8_Output renamed V1V8_OUTPUT
- net V3V3_Output renamed V3V3_OUTPUT
- net V5V_Input renamed V5V_INPUT
- net WiFi_nDisable renamed WIFI_NDISABLE
- net nRPIBOOT renamed N_RPIBOOT
