File: boards/DM0001/layout/layout.kicad_pcb (KiCad board)
At the start: 6 copper layers, 24.9 x 51.5 mm, 147 parts, among them IC1 TCAN330DCNT, IC2 LDFPVR, IC3 LDFPVR, IC4 L6387ED, IC5 L6387ED, IC6 L6387ED, IC7 STM32G431C8T6, J1 BM05B-SRSS-TB(LF)(SN), J2 BM05B-SRSS-TB(LF)(SN), J3 SM05B-SRSS-TB(LF)(SN), J4 ?, Q1 STL180N6F7, Q2 STL180N6F7, Q3 STL180N6F7, Q4 STL180N6F7, Q5 STL180N6F7, Q6 STL180N6F7, Y1 CSTNE8M00GH5C000R0

Commit message: chore(DM0001): update layout
Parts:
- L1: value LPS4018-333MRC -> ?
Other:
- board text added: "1.5660 mm"
- board text removed: "1.6000 mm"

Commit message: sync
Parts:
- added R17: ERJ-2RKF5232X, R_0402_1005Metric:R_0402_1005Metric, F.Cu at (92.4, 128.3)
- added R18: ERJ-2RKF4702X, R_0402_1005Metric:R_0402_1005Metric, F.Cu at (94.3, 129.3)
- C15, C17: value CL05A105KP5NNNC -> 1uF 10% 25V; moved to F.Cu
- C16, C18: value CL05A225MQ5NNNC -> 2.2uF 10% 16V; moved to F.Cu
- R13, R14: moved to F.Cu
- R15: value ERJ-2RKF1002X -> ERJ-2RKF4702X; moved to F.Cu
- R16: value ERJ-2RKF5232X -> ERJ-2RKF1002X; moved to F.Cu
- moved C18 27.1 mm to (96.2, 129.3), turned to 0 degrees
- moved C17 26.1 mm to (94.3, 128.3), turned to 0 degrees
- moved R15 21.0 mm to (92.4, 129.3), turned to 0 degrees
- moved R16 17.5 mm to (90.5, 127.3), turned to 0 degrees
- moved C16 15.6 mm to (92.4, 127.3), turned to 0 degrees
- moved C15 13.9 mm to (90.5, 126.3), turned to 0 degrees
- moved R13 13.2 mm to (90.5, 129.3), turned to 0 degrees
- moved R14 11.8 mm to (90.5, 128.3), turned to 0 degrees
- renumbered R17 to R19, R18 to R20, R19 to R21, R20 to R22, R21 to R23, R22 to R24, R23 to R25, R24 to R26, R25 to R27, R26 to R28, R27 to R29, R28 to R30, R29 to R31, R30 to R32, R31 to R33, R32 to R34, R33 to R35, R34 to R36, R35 to R37, R36 to R38, R37 to R39, R38 to R40, R39 to R41, R40 to R42, R41 to R43, R42 to R44, R43 to R45, R44 to R46, R45 to R47, R46 to R48, R47 to R49, R48 to R50, R49 to R51, R50 to R52, R51 to R53, R52 to R54, R53 to R55, R54 to R56, R55 to R57
Connections:
- net Ldo_3V3.ADJ_NC renamed Ldo_3V3._ADJ
- IC3 pad 2: Ldo_5V.ADJ_NC -> Ldo_5V._ADJ
- R15 pad 1: Ldo_5V.ADJ_NC -> Ldo_3V3.LDFPVR.NC_LDFPVR_PG
- R15 pad 2: GND -> V5V
- R16 pad 1: V5V -> Ldo_5V._ADJ
- R16 pad 2: Ldo_5V.ADJ_NC -> GND
Routing:
- net Ldo_5V._ADJ: track 0.00 -> 2.13 mm
- net Ldo_5V.ADJ_NC: track 2.13 -> 0.00 mm
