File: boards/Seward/layout/layout.kicad_pcb (KiCad board)
At the start: 4 copper layers, 40 x 14 mm, 34 parts, among them IC1 TPD4E05U06QDQARQ1, J1 ?, J2 FTSH-105-01-L-DV-K-A-P-TR, J3 USB4105-GF-A, SW1 B3U-1000P, U1 TPS74501PDRVR, U2 SN74LXC1T45DRYR, U3 SN74LXC1T45DRYR, U4 SN74LXC1T45DRYR, U5 STM32G0B1KBU6N

Commit message: layout(Seward): finalize board layout
Parts:
- moved C1 4.00 mm to (144.6, 102.2)
- moved C2 4.00 mm to (158.9, 104.0)
- moved C3 4.00 mm to (157.4, 97.2)
- moved C4 4.00 mm to (151.4, 94.6)
- moved C5 4.00 mm to (145.3, 94.3)
- moved C6 4.00 mm to (152.4, 94.6)
- moved C7 4.00 mm to (153.8, 99.5)
- moved C8 4.00 mm to (146.1, 99.0)
- moved D1 4.00 mm to (161.3, 96.0)
- moved D2 4.00 mm to (146.1, 96.5)
- moved D3 4.00 mm to (161.3, 94.8)
- moved D4 4.00 mm to (143.7, 95.7)
- moved IC1 4.00 mm to (143.7, 99.8)
- moved J1 4.00 mm to (146.0, 104.6)
- moved J2 4.00 mm to (161.6, 100.0)
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Routing:
- net GND: track 36.7 -> 38.6 mm, vias 19 -> 20
- net VTREF: track 23.1 -> 22.5 mm
- added copper zone on B.Cu, net VTREF
Other:
- board size 40 x 14 mm -> 32 x 14 mm
